Commit message: scale changed to 1 1 1 from 0.001

File: urdf/zbot.xacro (robot description, xacro)
@@ -20,5 +20,5 @@
     <origin xyz="0 0 0" rpy="0 0 0"/>
     <geometry>
-      <mesh filename="package://zbot_description/meshes/base_link.stl" scale="0.001 0.001 0.001"/>
+      <mesh filename="package://zbot_description/meshes/base_link.stl" scale="1 1 1"/>
     </geometry>
     <material name="silver"/>
@@ -27,5 +27,5 @@
     <origin xyz="0 0 0" rpy="0 0 0"/>
     <geometry>
-      <mesh filename="package://zbot_description/meshes/base_link.stl" scale="0.001 0.001 0.001"/>
+      <mesh filename="package://zbot_description/meshes/base_link.stl" scale="1 1 1"/>
     </geometry>
   </collision>
@@ -40,5 +40,5 @@
     <origin xyz="-0.049055 0.055 -0.005" rpy="0 0 0"/>
     <geometry>
-      <mesh filename="package://zbot_description/meshes/lb_wheel_1.stl" scale="0.001 0.001 0.001"/>
+      <mesh filename="package://zbot_description/meshes/lb_wheel_1.stl" scale="1 1 1"/>
     </geometry>
     <material name="silver"/>
@@ -47,5 +47,5 @@
     <origin xyz="-0.049055 0.055 -0.005" rpy="0 0 0"/>
     <geometry>
-      <mesh filename="package://zbot_description/meshes/lb_wheel_1.stl" scale="0.001 0.001 0.001"/>
+      <mesh filename="package://zbot_description/meshes/lb_wheel_1.stl" scale="1 1 1"/>
     </geometry>
   </collision>
@@ -60,5 +60,5 @@
     <origin xyz="0.049055 0.055 -0.005" rpy="0 0 0"/>
     <geometry>
-      <mesh filename="package://zbot_description/meshes/lf_wheel_1.stl" scale="0.001 0.001 0.001"/>
+      <mesh filename="package://zbot_description/meshes/lf_wheel_1.stl" scale="1 1 1"/>
     </geometry>
     <material name="silver"/>
@@ -67,5 +67,5 @@
     <origin xyz="0.049055 0.055 -0.005" rpy="0 0 0"/>
     <geometry>
-      <mesh filename="package://zbot_description/meshes/lf_wheel_1.stl" scale="0.001 0.001 0.001"/>
+      <mesh filename="package://zbot_description/meshes/lf_wheel_1.stl" scale="1 1 1"/>
     </geometry>
   </collision>
@@ -87,5 +87,5 @@
     <origin xyz="-0.049055 -0.055 -0.005" rpy="0 0 0"/>
     <geometry>
-      <mesh filename="package://zbot_description/meshes/rb_wheel_1.stl" scale="0.001 0.001 0.001"/>
+      <mesh filename="package://zbot_description/meshes/rb_wheel_1.stl" scale="1 1 1"/>
     </geometry>
     <material name="silver"/>
@@ -94,5 +94,5 @@
     <origin xyz="-0.049055 -0.055 -0.005" rpy="0 0 0"/>
     <geometry>
-      <mesh filename="package://zbot_description/meshes/rb_wheel_1.stl" scale="0.001 0.001 0.001"/>
+      <mesh filename="package://zbot_description/meshes/rb_wheel_1.stl" scale="1 1 1"/>
     </geometry>
   </collision>
@@ -107,5 +107,5 @@
     <origin xyz="0.049055 -0.055 -0.005" rpy="0 0 0"/>
     <geometry>
-      <mesh filename="package://zbot_description/meshes/rf_wheel_1.stl" scale="0.001 0.001 0.001"/>
+      <mesh filename="package://zbot_description/meshes/rf_wheel_1.stl" scale="1 1 1"/>
     </geometry>
     <material name="silver"/>
@@ -114,5 +114,5 @@
     <origin xyz="0.049055 -0.055 -0.005" rpy="0 0 0"/>
     <geometry>
-      <mesh filename="package://zbot_description/meshes/rf_wheel_1.stl" scale="0.001 0.001 0.001"/>
+      <mesh filename="package://zbot_description/meshes/rf_wheel_1.stl" scale="1 1 1"/>
     </geometry>
   </collision>
